File: PCB/Leiterkarte-v2.kicad_pcb (KiCad board)
At the start: 4 copper layers, 40.3 x 85.7 mm, 56 parts

Commit message: reorganization
Parts:
- removed RPM1: Conn_01x01_Pin, Connector_PinHeader_2.54mm:PinHeader_1x01_P2.54mm_Vertical
- added J1: B3B-XH-A, Hybrid_Dash:JST_B3B-XH-A, F.Cu at (224.7, 74.8)
- added J10: B2B-XH-A, Hybrid_Dash:JST_B2B-XH-A, F.Cu at (213.9, 111.3)
- added J2: B2B-XH-A, Hybrid_Dash:JST_B2B-XH-A, F.Cu at (213.9, 74.8)
- added J3: B3B-XH-A, Hybrid_Dash:JST_B3B-XH-A, F.Cu at (224.7, 82.1)
- added J4: B2B-XH-A, Hybrid_Dash:JST_B2B-XH-A, F.Cu at (213.9, 82.1)
- added J5: B3B-XH-A, Hybrid_Dash:JST_B3B-XH-A, F.Cu at (224.7, 89.4)
- added J6: B3B-XH-A, Hybrid_Dash:JST_B3B-XH-A, F.Cu at (224.7, 96.7)
- added J7: B2B-XH-A, Hybrid_Dash:JST_B2B-XH-A, F.Cu at (213.9, 89.4)
- added J8: B2B-XH-A, Hybrid_Dash:JST_B2B-XH-A, F.Cu at (213.9, 96.7)
- added J9: B2B-XH-A, Hybrid_Dash:JST_B2B-XH-A, F.Cu at (213.9, 104.0)
- added R3: 4.7k, Resistor_SMD:R_0603_1608Metric, F.Cu at (233.2, 72.5)
- added Rboot2: 10k, Resistor_SMD:R_0603_1608Metric, F.Cu at (233.2, 75.0)
- added Rboot3: 10k, Resistor_SMD:R_0603_1608Metric, F.Cu at (233.2, 77.5)
- added Rspd3: 10k, Resistor_SMD:R_0603_1608Metric, F.Cu at (233.2, 80.0)
- added Rspd4: 10k, Resistor_SMD:R_0603_1608Metric, F.Cu at (233.2, 82.5)
- added Rspd5: 10k, Resistor_SMD:R_0603_1608Metric, F.Cu at (233.2, 85.0)
- 3.3V1: footprint NCV33269DTRK3.3G:DPAK-3_ONS-M -> Hybrid_Dash:DPAK-3_ONS-M
- Cesp1: value 22uF -> 0.1uF
- Cesp2: value 0.1uF -> 22uF
- D1: value 550mV 5A -> B340A
- ESP_BOOT1, ESP_RST1: footprint button:small_button -> Hybrid_Dash:small_button
- L1: footprint SPM6530T:IND_SPM6530T-150M-HZ -> Hybrid_Dash:IND_SPM6530T-150M-HZ
- SD1: footprint MSD-1-A:CUI_MSD-1-A -> Hybrid_Dash:CUI_MSD-1-A
- USBC1: footprint USB-C 2.0:GCT_USB4105-GF-A -> Hybrid_Dash:GCT_USB4105-GF-A
- VRCond1: footprint MAX9924UAUB:SOP50P490X110-10N -> Hybrid_Dash:SOP50P490X110-10N
Connections:
- net BL renamed /blk
- net CLK renamed /clk
- net CS1 renamed /cs1
- net CS2 renamed /cs2
- net CS3 renamed /cs3
- net DC renamed /dc
- net DIN renamed /din
- net FANCTRL renamed /fan_control
- net Net-(ESP1-EN) renamed /enable
- net RIndicator renamed /r_indicator
- net RPM renamed /RPM_sense
- net RST renamed /rst
- net SD_CLK renamed /sd_clk
- net SD_CMD renamed /sd_cmd
- net SD_DAT0 renamed /sd_data0
- net SD_DAT1 renamed /sd_data1
- net SD_DAT2 renamed /sd_data2
- net SD_DAT3 renamed /sd_data3
- net Speed renamed /speed_sense
- net USB_D+ renamed /usb_d_pos
- net USB_D- renamed /usb_d_neg
- 5V1 pad 7: VCC -> Net-(5V1-VIN)
- Cin1 pad 1: VCC -> Net-(5V1-VIN)
- Cout1 pad 1: GND -> +3.3V
- Cout1 pad 2: +3.3V -> GND
- ESP1 pad 16: GND -> Net-(ESP1-IO46)
- ESP1 pad 20: Fuel -> /fuel_sense
- ESP1 pad 21: Oil -> /oil_sense
- ESP1 pad 22: WTemp -> /water_temp_sense
- ESP1 pad 24: TEMP2 -> unconnected-(ESP1-IO47-Pad24)
- ESP1 pad 26: GND -> Net-(ESP1-IO45)
- ESP1 pad 27: Net-(ESP1-IO0) -> /boot_mode
- ESP1 pad 33: TEMP1 -> /temp_sense
- ESP1 pad 34: LIndicator -> /l_indicator
- ESP1 pad 37: Button3 -> /button3_sense
- ESP1 pad 38: Button2 -> /button2_sense
- ESP1 pad 39: Button1 -> /button1_sense
- ESP_BOOT1 pad 2: Net-(ESP1-IO0) -> /boot_mode
- F1 pad 1: Net-(Vcc1-Pin_1) -> VCC
- F1 pad 2: VCC -> Net-(5V1-VIN)
- Qfan1 pad 3: Net-(Fan1-Pin_1) -> Net-(Qfan1-D)
- R1 pad 1: Net-(Speed1-Pin_2) -> Net-(J6-Pad3)
- R1 pad 2: Net-(VRCond1-IN-) -> Net-(VRCond1-IN+)
- R2 pad 1: Net-(Speed1-Pin_1) -> Net-(J6-Pad2)
- R2 pad 2: Net-(VRCond1-IN+) -> Net-(VRCond1-IN-)
- Rboot1 pad 1: Net-(ESP1-IO0) -> Net-(ESP1-IO46)
- Rboot1 pad 2: +3.3V -> GND
- Rfuel1 pad 1: +3.3V -> /fuel_sense
- Rfuel1 pad 2: Fuel -> +3.3V
- Rlind1 pad 1: Net-(Indics1-Pin_1) -> /l_indicator
- Rlind1 pad 2: LIndicator -> Net-(J4-Pad1)
- Rlind2 pad 1: LIndicator -> GND
- Rlind2 pad 2: GND -> /l_indicator
- Roil1 pad 1: +3.3V -> /oil_sense
- Roil1 pad 2: Oil -> +3.3V
- Rrind1 pad 1: Net-(Indics1-Pin_2) -> Net-(J4-Pad2)
- Rusb2 pad 1: Net-(USBC1-CC2) -> GND
- Rusb2 pad 2: GND -> Net-(USBC1-CC2)
- Rwtr1 pad 1: +3.3V -> /water_temp_sense
- Rwtr1 pad 2: WTemp -> +3.3V
- SPI1 pad 1: +5V -> +3.3V
- SPI2 pad 1: +5V -> +3.3V
- SPI3 pad 1: +5V -> +3.3V
Routing:
- net LIndicator: track 22.1 -> 0.00 mm
- net GND: track 70.0 -> 90.9 mm, vias 45 -> 44
- net VCC: track 14.1 -> 0.00 mm
- net Net-(5V1-VIN): track 0.00 -> 14.1 mm
- net /l_indicator: track 0.00 -> 1.21 mm, vias 0 -> 1
- net WTemp: vias 2 -> 0
- net Oil: vias 2 -> 0
- net Fuel: vias 2 -> 0
- net +3.3V: vias 6 -> 12
