File: PCB/Leiterkarte-v2.kicad_sch (KiCad schematic)
At the start: 39 parts

Commit message: reorganization
Parts:
- removed Buttons1: Conn_01x06_Pin, Connector_PinHeader_2.54mm:PinHeader_1x06_P2.54mm_Vertical, symbol Connector:Conn_01x06_Pin
- removed Fan1, Indics1, Speed1: Conn_01x02_Pin, Connector_JST:JST_SH_BM02B-SRSS-TB_1x02-1MP_P1.00mm_Vertical, symbol Connector:Conn_01x02_Pin
- removed GND1, RPM1, Vcc1: Conn_01x01_Pin, Connector_PinHeader_2.54mm:PinHeader_1x01_P2.54mm_Vertical, symbol Connector:Conn_01x01_Pin
- removed TEMP_S1, gauges1: Conn_01x03_Pin, Connector_JST:JST_SH_BM03B-SRSS-TB_1x03-1MP_P1.00mm_Vertical, symbol Connector:Conn_01x03_Pin
- removed TEMP_S2: MCP9700Ax-ETT, Package_TO_SOT_SMD:SOT-23, symbol Sensor_Temperature:MCP9700Ax-ETT
- added Cen1: 1uF, Capacitor_SMD:C_0805_2012Metric, symbol Device:C
- added Cesp1: 0.1uF, Capacitor_SMD:C_0805_2012Metric, symbol Device:C
- added Cesp2: 22uF, Capacitor_SMD:C_0805_2012Metric, symbol Device:C
- added Cshld1: 50nF, Capacitor_SMD:C_0805_2012Metric, symbol Device:C_Polarized
- added ESP1: ESP32-S3-WROOM-1U, RF_Module:ESP32-S3-WROOM-1U, symbol RF_Module:ESP32-S3-WROOM-1
- added ESP_BOOT1, ESP_RST1: SW_SPST, Hybrid_Dash:small_button, symbol Switch:SW_SPST
- added J1, J3, J5, J6: B3B-XH-A, Hybrid_Dash:JST_B3B-XH-A, symbol hybrid_dash_lib:B3B-XH-A
- added J10, J2, J4, J7, J8, J9: B2B-XH-A, Hybrid_Dash:JST_B2B-XH-A, symbol hybrid_dash_lib:B2B-XH-A
- added R3: 4.7k, Resistor_SMD:R_0603_1608Metric, symbol Device:R
- added Rboot1, Rboot2, Rboot3, Rspd3, Rspd4, Rspd5: 10k, Resistor_SMD:R_0603_1608Metric, symbol Device:R
- added Resp1, Rusb1, Rusb2: 5.1k, Resistor_SMD:R_0603_1608Metric, symbol Device:R
- added SD1: MSD-1-A, Hybrid_Dash:CUI_MSD-1-A, symbol MSD-1-A:MSD-1-A
- added SPI1, SPI2, SPI3: Conn_01x08, Connector_JST:JST_SH_BM08B-SRSS-TB_1x08-1MP_P1.00mm_Vertical, symbol Connector_Generic:Conn_01x08
- added USBC1: USB4105-GF-A, Hybrid_Dash:GCT_USB4105-GF-A, symbol USB-C:USB4105-GF-A
- 3.3V1: footprint NCV33269DTRK3.3G:DPAK-3_ONS-M -> Hybrid_Dash:DPAK-3_ONS-M
- D1: value 550mV 5A -> B340A
- L1: footprint SPM6530T:IND_SPM6530T-150M-HZ -> Hybrid_Dash:IND_SPM6530T-150M-HZ
- VRCond1: footprint MAX9924UAUB:SOP50P490X110-10N -> Hybrid_Dash:SOP50P490X110-10N
Connections:
- net Fuel is gone; now on net +3.3V: Rfuel1.2
- net Oil is gone; now on net +3.3V: Roil1.2
- net WTemp is gone; now on net +3.3V: Rwtr1.2
- net +3.3V: now also Cout1.1, Cesp1.1, Cesp2.1, ESP1.2 (3V3), J3.3, J5.3, J7.2, J8.2, J9.2, R3.1, Rboot3.1, Resp1.1, SD1.4 (VDD), SPI1.1 (Pin_1), SPI2.1 (Pin_1), SPI3.1 (Pin_1); no longer Cout1.2, Rfuel1.1, Roil1.1, Rwtr1.1
- net +5V: now also J10.2
- net GND: now also Cout1.2, Rlind2.1, Cen1.1, Cesp1.2, Cesp2.2, Cshld1.1, ESP1.1 (GND), ESP1.40 (GND), ESP1.41 (GND), ESP_BOOT1.1 (A), ESP_RST1.1 (A), J2.1, J3.2, J5.2, Rboot1.2, Rboot2.2, Rspd3.2, Rspd4.2, Rspd5.2, Rusb1.2, Rusb2.1, SD1.6 (VSS), SPI1.2 (Pin_2), SPI2.2 (Pin_2), SPI3.2 (Pin_2), USBC1.A1_B12 (GND), USBC1.B1_A12 (GND__1), USBC1.SH1 (SHELL_GND), USBC1.SH2 (SHELL_GND__1), USBC1.SH3 (SHELL_GND__2), USBC1.SH4 (SHELL_GND__3); no longer Cout1.1, Rlind2.2
- net VCC: now also F1.1, J2.2; no longer 5V1.7 (VIN), Cin1.1, F1.2
- net at Qfan1.3 (D): now also J10.1
- net l_indicator: now reaches Rlind1.1
- net l_indicator: now also Rlind2.2, ESP1.34 (IO41)
- net at Rrind1.1: now also J4.2
- net at R2.1: now also J6.2
- net at R1.1: now also J6.3
- net at Rrpm1.2: now also J6.1
- net at Cmax1.1, VRCond1.2 (IN-): now also R2.2; no longer R1.2
- net at Cmax1.2, VRCond1.1 (IN+): now also R1.2; no longer R2.2
- net FANCTRL renamed fan_control
- net fan_control: now also ESP1.36 (RXD0)
- net LIndicator: no longer names the net of Rlind1.2
- net LIndicator: now also J4.1; no longer Rlind2.1
- net RIndicator renamed r_indicator
- net r_indicator: now also ESP1.35 (IO42)
- net RPM renamed RPM_sense
- net RPM_sense: now also ESP1.23 (IO21)
- net Speed renamed speed_sense
- net speed_sense: now also ESP1.25 (IO48)
- new net: Rusb1.1, USBC1.A5 (CC1)
- new net: Rusb2.2, USBC1.B5 (CC2)
- new net: 5V1.7 (VIN), Cin1.1, F1.2
- new net: ESP1.16 (IO46), Rboot1.1
- new net: Cshld1.2, SD1.G1 (COVER_GND), SD1.G2 (COVER_GND), SD1.G3 (COVER_GND), SD1.G4 (COVER_GND)
- new net: ESP1.26 (IO45), Rboot2.1
- new net blk: ESP1.31 (IO38), SPI1.8 (Pin_8), SPI2.8 (Pin_8), SPI3.8 (Pin_8)
- new net boot_mode: ESP1.27 (IO0), ESP_BOOT1.2 (B), Rboot3.2
- new net button1_sense: ESP1.39 (IO1), J9.1, Rspd3.1
- new net button2_sense: ESP1.38 (IO2), J7.1, Rspd4.1
- new net button3_sense: ESP1.37 (TXD0), J8.1, Rspd5.1
- new net clk: ESP1.19 (IO11), SPI1.4 (Pin_4), SPI2.4 (Pin_4), SPI3.4 (Pin_4)
- new net cs1: ESP1.18 (IO10), SPI1.5 (Pin_5)
- new net cs2: ESP1.17 (IO9), SPI2.5 (Pin_5)
- new net cs3: ESP1.11 (IO18), SPI3.5 (Pin_5)
- new net dc: ESP1.12 (IO8), SPI1.6 (Pin_6), SPI2.6 (Pin_6), SPI3.6 (Pin_6)
- new net din: ESP1.10 (IO17), SPI1.3 (Pin_3), SPI2.3 (Pin_3), SPI3.3 (Pin_3)
- new net enable: Cen1.2, ESP1.3 (EN), ESP_RST1.2 (B), Resp1.2
- new net fuel_sense: ESP1.20 (IO12), J1.1, Rfuel1.1
- new net oil_sense: ESP1.21 (IO13), J1.2, Roil1.1
- new net rst: ESP1.32 (IO39), SPI1.7 (Pin_7), SPI2.7 (Pin_7), SPI3.7 (Pin_7)
- new net sd_clk: ESP1.6 (IO6), SD1.5 (CLK)
- new net sd_cmd: ESP1.7 (IO7), SD1.3 (CMD)
- new net sd_data0: ESP1.5 (IO5), SD1.7 (DAT0)
- new net sd_data1: ESP1.4 (IO4), SD1.8 (DAT1)
- new net sd_data2: ESP1.9 (IO16), SD1.1 (DAT2)
- new net sd_data3: ESP1.8 (IO15), SD1.2 (CD/DAT3)
- new net temp_sense: ESP1.33 (IO40), J3.1, J5.1, R3.2
- new net usb_d_neg: ESP1.13 (IO19), USBC1.A7 (DN1), USBC1.B7 (DN2)
- new net usb_d_pos: ESP1.14 (IO20), USBC1.A6 (DP1), USBC1.B6 (DP2)
- new net water_temp_sense: ESP1.22 (IO14), J1.3, Rwtr1.1
- no-connect marks 2 -> 11
Other:
- removed sheet MCU
- note added: "ESP32-S3"
- note added: "Guages"
- note added: "Indicators"
- note added: "Micro SD Card Holder"
- note added: "Programming Buttons"
- note added: "SPI Bus"
- note added: "USB C - for flashing"
- note added: "Use with DS18B20"
- note removed: "Converts VR Reluctant Sensor output to 5V Square Wave"
- note removed: "Fuel"
- note removed: "Needed Components: [- Added ; + Connected] + 3x SPI + 1x SWD + 1x SD MMC - SD Card + 3x Ohmmeter (Oil, Temp, Fuel) + 2x Frequency Measurement (Speed, RPM) + 2x Voltage Check (Indicator L/R) + Temperature Sensor (inside MCU) + Buttons + Fan connector + 3x LEDs (WiFi/Bluetooth Module)"
- note removed: "Oil"
- note removed: "Possibility to use a 5V fan if needed"
- note removed: "RPM Circuit"
- note removed: "Speed - VR Conditioner"
- note removed: "The STM32 allows 3.6V max. We only measure <500Hz, so this divider has no negative affects"
- note removed: "Using Mode A2 See Datasheet for more information!"
- note removed: "Water Temperature"
- moved on the sheet: 3.3V1, 5V1, Cboot1, Cin1, Cin2, Cout1, Cout2, D1, F1, L1, Qfan1, Rfbb1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
